File: fiddlesticks.kicad_sch (KiCad schematic)
At the start: 67 parts, among them J1 USB_C_Receptacle_USB2.0_16P, J2 Conn_01x04_Pin, J3 Conn_02x04_Counter_Clockwise, J4 Conn_01x04_Socket, J5 Conn_01x02_Pin, M1 Motor_DC, M2 Motor_DC, M3 Motor_DC, M4 Motor_DC, Q1 AO3400A, Q2 AO3400A, Q3 AO3400A, Q4 AO3400A, SW1 SW_Push, SW2 SW_SPDT, U1 STM32F411CEUx, U2 USBLC6-2SC6, U3 ICM-45605, U4 SPX3819M5-L-3-3, Y1 8MHz 18pF

Commit message: revised schematic
Parts:
- removed C7: 10u, Capacitor_SMD:C_0805_2012Metric_Pad1.18x1.45mm_HandSolder, symbol Device:C
- removed C8: 10n, Capacitor_SMD:C_0603_1608Metric_Pad1.08x0.95mm_HandSolder, symbol Device:C
- removed D10, D11, D12: PMEG2010AEH, Diode_SMD:D_SOD-123F, symbol Diode:PMEG2010AEH
- removed D3: RED, LED_SMD:LED_0805_2012Metric_Pad1.15x1.40mm_HandSolder, symbol Device:LED
- removed D5, D6, D7, D8: SS24, Diode_SMD:D_SMA, symbol Diode:SS24
- removed J3: Conn_02x04_Counter_Clockwise, Connector_PinHeader_2.54mm:PinHeader_2x08_P2.54mm_Vertical, symbol Connector_Generic:Conn_02x04_Counter_Clockwise
- removed J4: Conn_01x04_Socket, Connector_PinHeader_2.54mm:PinHeader_1x04_P2.54mm_Vertical, symbol Connector:Conn_01x04_Socket
- removed M1, M2, M3, M4: Motor_DC, symbol Motor:Motor_DC
- removed Q1, Q2, Q3, Q4: AO3400A, Package_TO_SOT_SMD:SOT-23, symbol Transistor_FET:AO3400A
- removed R14, R15, R16, R17: 33, Resistor_SMD:R_0805_2012Metric_Pad1.20x1.40mm_HandSolder, symbol Device:R
- removed R3, R4: 5.1K, Resistor_SMD:R_0805_2012Metric_Pad1.20x1.40mm_HandSolder, symbol Device:R
- removed SW2: SW_SPDT, symbol Switch:SW_SPDT
- removed U3: ICM-45605, IMU:XDCR_ICM-45605, symbol IMU:ICM-45605
- added C10, C11, C17, C18, C22, C24: 10u, symbol Device:C
- added C23: 100n, symbol Device:C
- added D3: ESD5Z3.3, Diode_SMD:D_SOD-523, symbol Diode:ESD5Zxx
- added D5, D6, D8: PMEG2010AEH, Diode_SMD:D_SOD-123F, symbol Diode:PMEG2010AEH
- added D7: RED, symbol Device:LED
- added FB1: 200 Ohms @ 100MHz, symbol Device:FerriteBead_Small
- added J3: Conn_01x04_Pin, symbol Connector:Conn_01x04_Pin
- added J4: Conn_02x04_Counter_Clockwise, symbol Connector_Generic:Conn_02x04_Counter_Clockwise
- added L1: 4.7uH, symbol Device:L
- added R10, R11: 0, symbol Device:R
- added SW2: SW_Push, symbol Switch:SW_Push
- added U3: MCP1640Bx-xCHY, Package_TO_SOT_SMD:SOT-23-6, symbol Regulator_Switching:MCP1640Bx-xCHY
- C12: value 4.7u -> 10u; footprint Capacitor_SMD:C_0805_2012Metric_Pad1.18x1.45mm_HandSolder -> (none)
- C13: footprint Capacitor_SMD:C_0805_2012Metric_Pad1.18x1.45mm_HandSolder -> (none); now not fitted
- C14: value 10u -> 4.7u; footprint Capacitor_SMD:C_0805_2012Metric_Pad1.18x1.45mm_HandSolder -> (none)
- C15: value 100n -> 10u; footprint Capacitor_SMD:C_0603_1608Metric_Pad1.08x0.95mm_HandSolder -> (none); now not fitted
- C16: value 100n -> 10n; footprint Capacitor_SMD:C_0603_1608Metric_Pad1.08x0.95mm_HandSolder -> (none)
- C19, C21: value 10u -> 100n; footprint Capacitor_SMD:C_0805_2012Metric_Pad1.18x1.45mm_HandSolder -> (none)
- C20: value 10u -> 100n; footprint Capacitor_SMD:C_0805_2012Metric_Pad1.18x1.45mm_HandSolder -> (none); now not fitted
- C6: renamed from C11; value 22pF -> 27pF
- C7: renamed from C10; value 22pF -> 27pF
- C9: value 100n -> 4.7u; footprint Capacitor_SMD:C_0603_1608Metric_Pad1.08x0.95mm_HandSolder -> (none)
- D1, D2, D4: value ESD5Zxx -> ESD5Z3.3
- J2: footprint Connector_PinHeader_2.54mm:PinHeader_1x04_P2.54mm_Horizontal -> (none)
- R1: value 10k -> 1k; footprint Resistor_SMD:R_0805_2012Metric_Pad1.20x1.40mm_HandSolder -> (none); now not fitted
- R2: value 1k -> 10K; footprint Resistor_SMD:R_0805_2012Metric_Pad1.20x1.40mm_HandSolder -> (none)
- R5, R6: value 47k -> 5.1k; footprint Resistor_SMD:R_0805_2012Metric_Pad1.20x1.40mm_HandSolder -> (none)
- R7: value 47k -> 976k; footprint Resistor_SMD:R_0805_2012Metric_Pad1.20x1.40mm_HandSolder -> (none)
- R8: value 47k -> 309k; footprint Resistor_SMD:R_0805_2012Metric_Pad1.20x1.40mm_HandSolder -> (none)
- R9: value 0 -> 1k; footprint Resistor_SMD:R_0805_2012Metric_Pad1.20x1.40mm_HandSolder -> (none)
- renumbered C18 to C8, R12 to R3, R13 to R4
Connections:
- net SW_BOOT0 is gone; now on net +3.3V: R1.1
- net +3.3V: now also C17.1, D7.2 (A), J4.8 (Pin_8), R10.1, SW2.1; no longer C1.2, C12.2, C13.2, C14.1, C14.2, C15.1, C15.2, C16.1, C16.2, C19.2, C2.2, C20.2, C21.2, C3.2, C4.2, C5.2, C6.2, C6.2, C7.1, C8.2, C9.2, D1.2 (A), D2.2 (A), D4.2 (A), J1.A1 (GND), J1.A12 (GND), J1.B1 (GND), J1.B12 (GND), J1.S1 (SHIELD), J2.3 (Pin_3), J5.2 (Pin_2), R2.1, R4.1, R5.2, R6.2, R7.2, R8.2, R9.2, SW1.1, U1.23 (VSS), U1.35 (VSS), U1.47 (VSS), U1.49 (VSS), U1.8 (VSSA), U2.2 (GND), U4.2 (GND)
- net +3.3VA: now also C19.1, C18.1, R10.2; no longer C6.1, R9.1
- net +5V: now also C23.1, C24.1, D6.2 (A), R11.2
- net RC_RX: now also J3.2 (Pin_2)
- net RC_TX: now also J3.1 (Pin_1)
- net SWCLK: now also D4.1 (K); no longer D2.1 (K)
- net SWDIO: now also D3.1 (K); no longer D1.1 (K)
- net VBAT: now also C12.1, C13.1, C14.1, C10.1, C11.1, D8.2 (A), L1.1, U3.3 (EN), U3.6 (V_{IN}); no longer C19.1, C20.1, C21.1
- net VBUS: now also D5.2 (A)
- net VSYS: now also C15.1, C21.1, C22.1, FB1.2; no longer C13.1, D9.1 (K)
- net at U4.4 (BP): now also C16.1
- net at U1.22 (VCAP1): now also C9.1; no longer C12.1
- net at J1.A5 (CC1): now also R5.1
- net at R7.1: now also R11.1, U3.5 (V_{OUT})
- net at R6.1: now also J1.B5 (CC2)
- net GND: now reaches R8.1
- net GND: now also C1.2, C12.2, C13.2, C14.2, C15.2, C16.2, C19.2, C2.2, C20.2, C21.2, C3.2, C4.2, C5.2, C6.2, C6.2, C7.1, C8.2, C9.2, D1.2 (A), D2.2 (A), D4.2 (A), J1.A1 (GND), J1.A12 (GND), J1.B1 (GND), J1.B12 (GND), J1.S1 (SHIELD), J2.3 (Pin_3), J5.2 (Pin_2), R2.2, R4.1, R5.2, R6.2, R9.1, SW1.1, U2.2 (GND), U4.2 (GND), C10.2, C11.2, C17.2, C18.2, C22.2, C23.2, C24.2, D3.2 (A), J3.4 (Pin_4), J4.1 (Pin_1), U3.2 (GND)
- net mcu_boot0: now reaches U1.44 (BOOT0)
- net mcu_boot0: now also D2.1 (K), R2.1, SW2.2; no longer R1.2
- net BAT_ADC1 renamed LiPo_ADC1
- net Din+ renamed DIN+
- net Din- renamed DIN-
- net NRST renamed mcu_nrst
- net mcu_nrst: now also C6.1, D1.1 (K), R1.2; no longer C9.1, D4.1 (K)
- net nrf_ce renamed NRF_CE
- net NRF_CE: now also J4.2 (Pin_2)
- net nrf_miso renamed NRF_MISO
- net NRF_MISO: now also J4.4 (Pin_4)
- net nrf_mosi renamed NRF_MOSI
- net NRF_MOSI: now also J4.6 (Pin_6)
- net nrf_ncs renamed NRF_NCS
- net NRF_NCS: now also J4.7 (Pin_7)
- net nrf_sck renamed NRF_SCK
- net NRF_SCK: now also J4.3 (Pin_3)
- net pwm1 renamed motor_driver_imu/PWM1
- net pwm2 renamed motor_driver_imu/PWM2
- net pwm3 renamed motor_driver_imu/PWM3
- net pwm4 renamed motor_driver_imu/PWM4
- new net: D5.1 (K), D6.1 (K), J3.3 (Pin_3)
- new net: D7.1 (K), R9.2
- new net: C20.1, D8.1 (K), D9.1 (K), FB1.1
- new net: R7.2, R8.2, U3.4 (V_{FB})
- new net: U1.23 (VSS), U1.35 (VSS), U1.47 (VSS), U1.49 (VSS)
- new net: L1.2, U3.1 (SW)
- no-connect marks 16 -> 4
Other:
- removed sheet VBAT_to_5V
- added sheet motor_driver_imu (motor_driver_imu.kicad_sch)
- note added: "1.21V"
- note added: "3.3V low noise LDO"
- note added: "5V Boost converter for external RX"
- note added: "BOOT0"
- note added: "BT2.0 male connector"
- note added: "External RX Pads"
- note added: "FiddleSticks FlightController"
- note added: "LiPo (1s1p 4.2V Input pad)"
- note added: "NRF24l01+ external board used as backup"
- note added: "NRST"
- note added: "Power OR between VBUS and VBAT"
- note added: "SWDIO header pins"
- note added: "Target Dim: 50x50 (mm) Target Weight: < 70 ( g)"
- note added: "USB ESD Protection"
- note added: "USB Peripheral"
- note added: "VDDA use ferrite if needed"
- note added: "filter if noise is too high"
- note removed: "BT2.0 male connector for battery"
- note removed: "I'll use Ferrite bead if i really need to"
- note removed: "Motor Drivers"
- note removed: "Note that nrf24l01 will only be used as fallback incase i dont have a UART supported receiver"
- note removed: "Receiver pads"
- note removed: "fiddlesticks drone"
- note removed: "supports only 1s1p 4.35 LiPo"
- note removed: "target dimensions 50x50 (mm) target weight < 70g"
- moved on the sheet: C1, C2, C3, C4, C5, C6, C7, C8, D1, J1, R3, R4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
